File: versions/v0.1/_autosave-CCC_ESC.kicad_sch (KiCad schematic)
At the start: 160 parts, among them J1 Conn_01x04, J2 Conn_01x06, J3 Conn_01x06, J4 Conn_01x06, SW1 Conn_01x02, U1 NCP5183, U2 NCP5183, U3 NCP5183, U4 NCS20074D, U5 STM32F401CCU6_Balckpill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

Commit message: minor rerouting
Parts:
- gave numbers to parts that had none: 1
Changed lines of the file:
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@@
   (symbol (lib_id "CCC_ESC_Custom_Symbols:TO220_replacement_module") (at 166.37 76.2 0) (unit 1)
     (in_bom yes) (on_board yes) (fields_autoplaced)
-    (property "Reference" "U?" (id 0) (at 175.895 71.12 0))
+    (property "Reference" "U8" (id 0) (at 175.895 71.12 0))
     (property "Value" "TO220_replacement_module" (id 1) (at 175.895 73.66 0))
     (property "Footprint" "CCC_ESC_Custom_parts:TO220_replacement_module" (id 2) (at 166.37 76.2 0)
@@
   (symbol (lib_id "power:GND") (at 172.72 91.44 0) (unit 1)
     (in_bom yes) (on_board yes) (fields_autoplaced)
-    (property "Reference" "#PWR?" (id 0) (at 172.72 97.79 0)
+    (property "Reference" "#PWR0128" (id 0) (at 172.72 97.79 0)
       (effects (font (size 1.27 1.27)) hide)
     )
@@
       (reference "#PWR0127") (unit 1) (value "GND") (footprint "")
     )
+    (path "/d02bdb00-0af7-4a63-8ecd-9e921ab6b466"
+      (reference "#PWR0128") (unit 1) (value "GND") (footprint "")
+    )
     (path "/894703c7-10d0-472a-bf81-33f567b69f44"
       (reference "#PWR0132") (unit 1) (value "GND") (footprint "")
@@
       (reference "#PWR0137") (unit 1) (value "GND") (footprint "")
     )
-    (path "/d02bdb00-0af7-4a63-8ecd-9e921ab6b466"
-      (reference "#PWR?") (unit 1) (value "GND") (footprint "")
-    )
     (path "/c5bdcfd4-44ee-4a47-b511-8d607870eba8"
       (reference "C1") (unit 1) (value "10uF") (footprint "Capacitor_SMD:C_0603_1608Metric")
@@
     )
     (path "/68236c93-49e7-4933-ab0e-48bd3cb739ea"
-      (reference "U?") (unit 1) (value "TO220_replacement_module") (footprint "CCC_ESC_Custom_parts:TO220_replacement_module")
-    )
-  )
+      (reference "U8") (unit 1) (value "TO220_replacement_module") (footprint "CCC_ESC_Custom_parts:TO220_replacement_module")
+    )
+  )
