File: versions/v0.1/_autosave-CCC_ESC.kicad_sch (KiCad schematic)
At the start: 176 parts, among them J1 Conn_01x04, J2 Conn_01x06, J3 Conn_01x06, J4 Conn_01x06, SW1 Conn_01x02, U1 NCP5183, U2 NCP5183, U3 NCP5183, U4 NCS20074D, U5 STM32F401CCU6_Balckpill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

Commit message: phase nodes redesigned
Parts:
- gave numbers to parts that had none: 3
Changed lines of the file:
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@@
   (symbol (lib_id "Connector:TestPoint") (at 541.0552 241.3 0) (unit 1)
     (in_bom yes) (on_board yes)
-    (property "Reference" "PH?" (id 0) (at 541.02 236.22 0)
+    (property "Reference" "PH8" (id 0) (at 541.02 236.22 0)
       (effects (font (size 1.27 1.27)) (justify left))
     )
@@
   (symbol (lib_id "Connector:TestPoint") (at 538.48 241.3 0) (unit 1)
     (in_bom yes) (on_board yes)
-    (property "Reference" "PH?" (id 0) (at 537.21 236.22 0)
+    (property "Reference" "PH7" (id 0) (at 537.21 236.22 0)
       (effects (font (size 1.27 1.27)) (justify left))
     )
@@
   (symbol (lib_id "Connector:TestPoint") (at 543.56 241.3 0) (unit 1)
     (in_bom yes) (on_board yes)
-    (property "Reference" "PH?" (id 0) (at 544.83 236.22 0)
+    (property "Reference" "PH9" (id 0) (at 544.83 236.22 0)
       (effects (font (size 1.27 1.27)) (justify left))
     )
@@
       (reference "PH6") (unit 1) (value "PhasePad") (footprint "TestPoint:TestPoint_THTPad_D4.0mm_Drill2.0mm")
     )
-    (path "/59695976-f92b-47f0-b0bc-f405b8ef41ca"
-      (reference "PH?") (unit 1) (value "PhasePad") (footprint "TestPoint:TestPoint_THTPad_D4.0mm_Drill2.0mm")
-    )
     (path "/811e104a-3ed6-4432-80de-7f1b4d60e609"
-      (reference "PH?") (unit 1) (value "PhasePad") (footprint "TestPoint:TestPoint_THTPad_D4.0mm_Drill2.0mm")
+      (reference "PH7") (unit 1) (value "PhasePad") (footprint "TestPoint:TestPoint_THTPad_D4.0mm_Drill2.0mm")
+    )
+    (path "/59695976-f92b-47f0-b0bc-f405b8ef41ca"
+      (reference "PH8") (unit 1) (value "PhasePad") (footprint "TestPoint:TestPoint_THTPad_D4.0mm_Drill2.0mm")
     )
     (path "/a9f8a06b-6dbe-4bc7-9d27-22fb33fac9e6"
-      (reference "PH?") (unit 1) (value "PhasePad") (footprint "TestPoint:TestPoint_THTPad_D4.0mm_Drill2.0mm")
+      (reference "PH9") (unit 1) (value "PhasePad") (footprint "TestPoint:TestPoint_THTPad_D4.0mm_Drill2.0mm")
     )
     (path "/155a305d-cff1-4340-986a-f6393f0cc554"
